File: OctaveEnv.kicad_pcb (KiCad board)
At the start: 4 copper layers, 100 x 65 mm, 91 parts, among them J101 IN, J102 PWR, J103 OUT, Q101 BC857, SW101 Stomp, U101 AZ34063U, U102 L7805, U103 TL074, U104 74HCT74, U105 LM13700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

Commit message: octave up sim
Parts:
- POT101: value 100kB -> 10kB
- POT103: value 100kB -> 1MB
- POT104: value 100kB -> 50kB
- R113: value 22k -> 220k
- R119: value 33k -> 330k
Changed lines of the file:
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@@
 			)
 		)
-		(property "Value" "22k"
+		(property "Value" "220k"
 			(at 0 1.65 0)
 			(layer "F.Fab")
@@
 			)
 		)
-		(property "Value" "100kB"
+		(property "Value" "10kB"
 			(at 0 9.86 90)
 			(layer "F.Fab")
@@
 			)
 		)
-		(property "Value" "100kB"
+		(property "Value" "50kB"
 			(at 0 9.86 90)
 			(layer "F.Fab")
@@
 			)
 		)
-		(property "Value" "33k"
+		(property "Value" "330k"
 			(at 0 1.65 0)
 			(layer "F.Fab")
@@
 			)
 		)
-		(property "Value" "100kB"
+		(property "Value" "1MB"
 			(at 0 9.86 90)
 			(layer "F.Fab")
@@
 		(tags "test point THT pad")
 		(property "Reference" "TP108"
-			(at 0 1.648 360)
+			(at 0 1.648 0)
 			(layer "B.SilkS")
 			(hide yes)
@@
 		)
 		(property "Value" "SWC"
-			(at 0 -1.75 360)
+			(at 0 -1.75 0)
 			(layer "B.SilkS")
 			(effects
@@
 		)
 		(fp_text user "${REFERENCE}"
-			(at 0 1.65 360)
+			(at 0 1.65 0)
 			(layer "B.Fab")
 			(effects
